File: Hardware/Three_Phase_Inverter_Controller.sch (KiCad schematic (older format))
At the start: 78 parts

Commit message: renamed project. Added more datasheets
Parts:
- removed U?: FT230XS, symbol FT230XS-RESCUE-EV_FET_DRIVER
- added U?: FT230XS, symbol FT230XS
Other:
- moved on the sheet: C?, U?

Commit message: Updated schematic
Parts:
- removed D? (x2): LED, symbol LED_ALT
- removed Q? (x2): VAL, symbol Q_NMOS_GSD
- removed R? (x2): 10K, symbol R_Small
- removed R? (x2): 470R, symbol R_Small
- added AA? (x2): OUT_1_H, symbol TEST_1P
- added AA? (x2): OUT_1_L, symbol TEST_1P
- added C?: 4.5nF, symbol C_Small
- added C? (x5): 100nF, symbol C_Small
- added C? (x4): 4.7uF, symbol C_Small
- added D? (x2): VAL, symbol D_Schottky_Small_ALT
- added J?: ISP, symbol CONN_02X03
- added J?: I2C, symbol CONN_01X03
- added J?: SPARE, symbol CONN_01X04
- added J?: EXT_IN, symbol CONN_01X10
- added JP?: SHDN_SELECT, symbol Jumper_NC_Dual
- added Q? (x4): IXFN110N60P3, symbol Q_NMOS_GSD
- added R?: 1M, symbol R_Small
- added R? (x9): 10K, symbol R_Small
- added R? (x4): 10R, symbol R_Small
- added SW?: ~MCU_RST, symbol SW_PUSH
- added TVS?: PRTR5V0U2X, symbol PRTR5V0U2X
- added U? (x2): IR2110S, symbol IR2110S
Connections:
- net labels added: BLU_DRVH, BLU_DRVH_R, BLU_DRVL, BLU_DRVL_R, BLU_VB, BLU_VS, EX_SD/SCK, GRN_DRVH, GRN_DRVH_R, GRN_DRVL, GRN_DRVL_R, GRN_VB, GRN_VS, MODE/MOSI, M_SD/MISO, PB4/MISO, PB7, PE2, PE3, SD, SHDN/SCK
- net labels removed: DRV_SHDN, I2C, MODE
- wire segments 331 -> 511
Other:
- note added: "BLUE_OUT"
- note added: "GREEN_OUT"
- moved on the sheet: C?, D?, J?, L?, Q?, R?, TP?, U?
