File: Hardware/Three_Phase_Inverter_Controller.sch (KiCad schematic (older format))
At the start: 113 parts

Commit message: Added Diode OR to Power Supply
Parts:
- added C? (x4): 4.7uF, symbol C_Small
- added U?: LTC4413, symbol LTC4413
Connections:
- net +5V: now also C?.1, C?.1, C?.1, U?.1 (INA), U?.10 (OUTA), U?.6 (OUTB)
- net GND: now also C?.2, C?.2, C?.2, C?.2, U?.11 (GND), U?.2 (~ENBA), U?.3 (GND), U?.4 (~ENBB)
- new net: C?.1, U?.5 (INB)
- no-connect marks 3 -> 4
Other:
- moved on the sheet: C?, D?, J?, JP?, L?, Q?, R?, SW?, TP?, TVS?, U?

Commit message: Annotated schematic
Parts:
- gave numbers to parts that had none: 118
Other:
- moved on the sheet: C1, C10, C11, C12, C13, C14, C15, C16, C17, C18, C19, C2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

Commit message: Pre-release v0.3 Schematic
Parts:
- removed J2: EXT_IN, symbol CONN_01X10
- added J1: UART, symbol CONN_01X03
- added J3: HALL, symbol CONN_01X04
- added J4: CURRENT, symbol CONN_01X08
- added JP1: I2C_SDA, symbol Jumper
- added JP2: I2C_SCL, symbol Jumper
- added R2, R20, R21, R29, R3, R4: 10K, symbol R_Small
- renumbered J1 to J2, J3 to J5, J4 to J6, J5 to J7, J6 to J8, JP1 to JP3, R7 to R10, R8 to R11, R9 to R12, R10 to R13, R11 to R14, R12 to R15, R13 to R16, R14 to R17, R15 to R18, R16 to R19, R17 to R22, R18 to R23, R19 to R24, R20 to R25, R21 to R26, R22 to R27, R23 to R28, R24 to R30, R25 to R31, R26 to R32, R27 to R33, R28 to R34, R29 to R35, R30 to R36, R31 to R37, R32 to R38, R33 to R39, R34 to R40, R35 to R41, R2 to R5, R3 to R7, R4 to R8, R5 to R9
Connections:
- net AREF is gone; now on net +5V: R18.2, R19.1, R22.2, U5.3 (+)
- net +5V: now also R2.2, R20.2, R21.2, R29.2, R3.2, R4.2
- net CMD_CURR0: now also J4.5 (P5)
- net CMD_CURR1: now also J4.4 (P4)
- net CMD_CURR2: now also J4.3 (P3)
- net CMD_CURR3: now also J4.2 (P2)
- net CMD_CURR4: now also J4.1 (P1)
- net GND: now also J1.1 (P1), J3.1 (P1), J4.6 (P6), J4.8 (P8)
- net I2C_SCL: now also JP2.1; no longer R10.1, R11.1
- net I2C_SDA: now also JP1.1; no longer R5.1, R6.1
- net LINK_CURR: now also J4.7 (P7)
- net POS_A: now also J3.4 (P4), R2.1
- net POS_B: now also J3.3 (P3), R3.1
- net POS_C: now also J3.2 (P2), R4.1
- net RXD: now also J1.2 (P2), R20.1
- net SD: now also R29.1
- net TXD: now also J1.3 (P3), R21.1
- net VBUS_DET: now also R7.1, R8.2; no longer R8.1, R9.2
- new net: R8.1, R9.2
- new net: JP1.2, R5.1, R6.1
- new net: JP2.2, R10.1, R11.1
Other:
- moved on the sheet: C1, C10, C11, C12, C13, C14, C15, C16, C17, C18, C19, C2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

Commit message: Update to pre-release v0.4
Parts:
- removed R20: 10K, symbol R_Small
- added C43: 27pF, symbol C_Small
- added C8: 100nF, symbol C_Small
- added JP2: HALL, symbol Jumper
- added JP4: SD, symbol Jumper
- added R12, R13, R14, R15: 0R, symbol R_Small
- added R45: 0.05R, symbol R_Small
- added R46: 10k, symbol R_Small
- added TP?: +12V, symbol TEST
- added TP?: 12V_HLDP, symbol TEST
- added TP?: 5V_BUCK, symbol TEST
- added TP?: VIN, symbol TEST
- C21: renamed from C22; value VAL -> 4.7uF
- C3, C4, C5: value VAL -> 150uF
- D1, D2, D4, D5, D6: value VAL -> PMEG6030ETP
- JP1: value I2C_SDA -> HALL
- L1: value VAL -> 68uH
- R16: renamed from R14; value VAL -> 0R
- R17: renamed from R15; value VAL -> 45.3k
- R25: renamed from R23; value VAL -> 68k
- R26: renamed from R24; value VAL -> 12k
- renumbered C12 to C10, C14 to C11, C7 to C12, C18 to C13, C10 to C14, C11 to C15, C20 to C16, C13 to C17, C15 to C18, C21 to C19, C16 to C20, C17 to C22, C19 to C23, C23 to C24, C24 to C27, C27 to C30, C30 to C31, C31 to C32, C32 to C33, C33 to C34, C34 to C35, C35 to C36, C36 to C37, C37 to C38, C38 to C39, C39 to C40, C40 to C41, C41 to C42, C8 to C7, J2 to J1, J3 to J2, J4 to J3, J5 to J4, J6 to J5, J1 to J6, JP2 to JP3, JP3 to JP5, R16 to R18, R17 to R19, R12 to R20, R13 to R21, R18 to R22, R19 to R23, R22 to R24, R25 to R27, R21 to R28, R27 to R29, R28 to R30, R26 to R31, R29 to R32, R30 to R33, R31 to R34, R32 to R35, R33 to R36, R34 to R37, R35 to R38, R36 to R39, R37 to R40, R38 to R41, R39 to R42, R40 to R43, R41 to R44, U3 to U2, U5 to U3, U2 to U4, U4 to U5, U8 to U7, U7 to U8
Connections:
- net +12V: now also R45.1, TP?.1, TP?.1; no longer J1.2 (P2)
- net +5V: now also JP1.2, C43.1, C8.1, R14.2, R46.1, TP?.1, TP?.1; no longer R2.2, R3.2, R4.2
- net BUCK_FB: now also C43.2
- net GND: now also C8.2, R15.2, R46.2
- net I2C_SCL: now also R13.2; no longer U5.6 (PE1(PTCXY/SCL1/T4))
- net I2C_SDA: now also JP2.1, R12.2; no longer JP1.1, U5.3 (PE0(PTCXY/SDA1/ICP4/ACO))
- net SD: now also JP4.2; no longer R32.1
- net at R5.1, R6.1: now also JP2.2; no longer JP1.2
- new net: JP1.1, R2.2, R3.2, R4.2
- new net: JP4.1, R32.1
- new net PE0: R12.1, R15.1, U5.3 (PE0(PTCXY/SDA1/ICP4/ACO))
- new net PE1: R13.1, R14.1, U5.6 (PE1(PTCXY/SCL1/T4))
- new net VIN: J1.2 (P2), R45.2
Other:
- note added: "ATMEGA328P/PB STRAPPING"
- note added: "ATMEGA328P: R12, R13 = DNP\nATMEGA328PB: C8, R14, R15 = DNP\n\nDEFAULT CONFIG: ATMEGA328PB"
- moved on the sheet: C1, C12, C14, C15, C17, C18, C2, C20, C21, C22, C23, C24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

Commit message: Updated BOM & finished SCH
Parts:
- D3: value LED_Dual -> LNJ167W8RRA
- R10, R11, R2, R28, R3, R31, R32, R4, R40, R41, R42, R43, R44, R5, R6, R7, R8, R9: value 10K -> 10k
- R18: value VAL -> 26.1k
- R19, R23: value VAL -> 10k
- R22: value VAL -> 6.8k
- R24: value VAL -> 470k
- R29, R30: value VAL -> 180R
- R3k: renamed from R39; value 10K -> 10k
- gave numbers to parts that had none: 4
Connections:
- net +5V: no longer R22.2, R23.1, R24.2, U3.3 (+)
- new net AREF: R22.2, R23.1, R24.2, U3.3 (+)
Other:
- note added: "Trip point (Low to High): 10.628 VDC (12V_HLDP)\nTrip point (High to Low): 10.773 VDC (12V_HLDP)"
- moved on the sheet: D3, R29, R30, U6

Commit message: Updated schematic
Parts:
- JP1: value HALL -> HALL_P_EN
- JP2: value HALL -> I2C_SDA
Changed lines of the file:
@@
 P 2900 6350
 F 0 "JP1" V 2946 6263 50  0000 R CNN
-F 1 "HALL" V 2855 6263 50  0000 R CNN
+F 1 "HALL_P_EN" V 2855 6263 50  0000 R CNN
 F 2 "" H 2900 6350 50  0001 C CNN
 F 3 "" H 2900 6350 50  0001 C CNN
@@
 P 4050 9375
 F 0 "JP2" V 4096 9288 50  0000 R CNN
-F 1 "HALL" V 4005 9288 50  0000 R CNN
+F 1 "I2C_SDA" V 4005 9288 50  0000 R CNN
 F 2 "" H 4050 9375 50  0001 C CNN
 F 3 "" H 4050 9375 50  0001 C CNN

Commit message: Assigned footrpints for most components, tweaked BOM
Parts:
- removed J4: I2C, symbol CONN_01X03
- removed J6: UART, symbol CONN_01X03
- added C44: 100nF, Capacitors_SMD:C_0603, symbol C_Small
- added J4: I2C, Pin_Headers:Pin_Header_Angled_1x04_Pitch2.54mm, symbol CONN_01X04
- added J6: UART, Pin_Headers:Pin_Header_Angled_1x04_Pitch2.54mm, symbol CONN_01X04
- C1, C10, C11, C12, C13, C15, C16, C17, C18, C19, C2, C22, C23, C24, C27, C30, C31, C32, C33, C40, C41, C42, C43, C6, C8, C9: footprint (none) -> Capacitors_SMD:C_0603
- C14, C20, C21, C25, C26, C28, C29, C34, C35, C36, C37, C38, C39, C7: footprint (none) -> Capacitors_SMD:C_1206
- C3, C4, C5: footprint (none) -> Capacitors_SMD:CP_Elec_10x10.5
- J1: footprint (none) -> Pin_Headers:Pin_Header_Angled_1x02_Pitch2.54mm
- J2: footprint (none) -> Pin_Headers:Pin_Header_Straight_1x04_Pitch2.54mm
- J3: footprint (none) -> Pin_Headers:Pin_Header_Angled_1x08_Pitch2.54mm
- J5: footprint (none) -> Pin_Headers:Pin_Header_Angled_1x04_Pitch2.54mm
- J8: footprint (none) -> Pin_Headers:Pin_Header_Straight_2x03_Pitch2.54mm
- JP1, JP2, JP3, JP4: footprint (none) -> Pin_Headers:Pin_Header_Straight_2x01_Pitch2.00mm
- JP5: footprint (none) -> Pin_Headers:Pin_Header_Straight_1x03_Pitch2.54mm
- R1, R10, R11, R12, R13, R14, R15, R16, R17, R18, R19, R2, R20, R21, R22, R23, R24, R25, R26, R27, R28, R3, R31, R32, R4, R40, R41, R42, R43, R44, R46, R5, R6, R7, R8, R9: footprint (none) -> Resistors_SMD:R_0603
- R29, R30, R33, R34, R35, R36, R37, R38: footprint (none) -> Resistors_SMD:R_0805
- R3k1: renamed from R3k; footprint (none) -> Resistors_SMD:R_0603
- R45: footprint (none) -> Resistors_SMD:R_1206
- SW1: footprint (none) -> Buttons_Switches_SMD:SW_SPST_TL3342
- TP1, TP2, TP3, TP4, TP5, TP6, TP7: footprint (none) -> Measurement_Points:Test_Point_Keystone_5019_Minature
- TVS1: footprint (none) -> TO_SOT_Packages_SMD:SOT-143
- U1: footprint (none) -> TO_SOT_Packages_SMD:SOT-23-6
- U2: footprint (none) -> Housings_SOIC:SOIC-8-1EP_3.9x4.9mm_Pitch1.27mm
- U3, U6: footprint (none) -> TO_SOT_Packages_SMD:SOT-23-5
- U4: footprint (none) -> Housings_SSOP:SSOP-16_3.9x4.9mm_Pitch0.635mm
- U7: footprint (none) -> Housings_DFN_QFN:DFN-8-1EP_3x3mm_Pitch0.5mm
- U8: footprint (none) -> Oscillators:Oscillator_SMD_EuroQuartz_XO53-4pin_5.0x3.2mm
Connections:
- net +5V: now also C26.1, U7.5 (INB), C44.1
- net GND: now also C44.2, J4.1 (P1), J4.4 (P4), J6.1 (P1), J6.4 (P4)
- net I2C_SCL: now also J4.2 (P2)
- net I2C_SDA: now also J4.3 (P3)
- net RXD: now also J6.2 (P2)
- net TXD: now also J6.3 (P3)
Other:
- moved on the sheet: R7, R8, R9

Commit message: Changed connector, started layout, save before reloading new netlist
Parts:
- removed J3: CURRENT, Pin_Headers:Pin_Header_Angled_1x08_Pitch2.54mm, symbol CONN_01X08
- removed J4: I2C, Pin_Headers:Pin_Header_Angled_1x04_Pitch2.54mm, symbol CONN_01X04
- removed J5: SPARE, Pin_Headers:Pin_Header_Angled_1x04_Pitch2.54mm, symbol CONN_01X04
- added J3: IN/I2C, symbol CONN_02X08
- added TP10: GRN_H, Measurement_Points:Test_Point_Keystone_5019_Minature, symbol TEST
- added TP11: GRN_L, Measurement_Points:Test_Point_Keystone_5019_Minature, symbol TEST
- added TP12: BLU_H, Measurement_Points:Test_Point_Keystone_5019_Minature, symbol TEST
- added TP13: BLU_L, Measurement_Points:Test_Point_Keystone_5019_Minature, symbol TEST
- added TP14: YLW_DRVH, Measurement_Points:Test_Point_Keystone_5019_Minature, symbol TEST
- added TP15: YLW_DRVL, Measurement_Points:Test_Point_Keystone_5019_Minature, symbol TEST
- added TP16: GRN_DRVH, Measurement_Points:Test_Point_Keystone_5019_Minature, symbol TEST
- added TP17: GRN_DRVL, Measurement_Points:Test_Point_Keystone_5019_Minature, symbol TEST
- added TP18: BLU_DRVH, Measurement_Points:Test_Point_Keystone_5019_Minature, symbol TEST
- added TP19: BLU_DRVL, Measurement_Points:Test_Point_Keystone_5019_Minature, symbol TEST
- added TP8: YLW_H, Measurement_Points:Test_Point_Keystone_5019_Minature, symbol TEST
- added TP9: YLW_L, Measurement_Points:Test_Point_Keystone_5019_Minature, symbol TEST
- D1, D2, D4, D5, D6: footprint (none) -> FritzLib:SOD-128
- J1: footprint Pin_Headers:Pin_Header_Angled_1x02_Pitch2.54mm -> Connectors_Terminal_Blocks:TerminalBlock_Pheonix_MPT-2.54mm_2pol
- J2: footprint Pin_Headers:Pin_Header_Straight_1x04_Pitch2.54mm -> Connectors_Terminal_Blocks:TerminalBlock_Pheonix_MPT-2.54mm_4pol
- J5: renamed from J7; footprint (none) -> FritzLib:USB-B_62910416121
- Q1, Q2, Q3, Q4, Q5, Q6: footprint (none) -> FritzLib:M4_SCREW_OFFSET_9.5_16ths
- U10, U11, U9: footprint (none) -> Housings_SOIC:SOIC-16W_7.5x10.3mm_Pitch1.27mm
- renumbered J6 to J4, J8 to J6
Connections:
- net BLU_DRVH_R: now also TP18.1
- net BLU_DRVL_R: now also TP19.1
- net BLU_H: now also TP12.1
- net BLU_L: now also TP13.1
- net CMD_CURR0: now also J3.8 (P8)
- net CMD_CURR1: now also J3.10 (P10)
- net CMD_CURR2: now also J3.12 (P12)
- net CMD_CURR3: now also J3.14 (P14)
- net CMD_CURR4: now also J3.16 (P16)
- net GND: now also J3.1 (P1), J3.2 (P2), J3.3 (P3), J3.5 (P5), J3.6 (P6)
- net GRN_DRVH_R: now also TP16.1
- net GRN_DRVL_R: now also TP17.1
- net GRN_H: now also TP10.1
- net GRN_L: now also TP11.1
- net I2C_SCL: now also JP2.1, R12.2, J3.15 (P15); no longer JP3.1, R13.2
- net I2C_SDA: now also JP3.1, R13.2, J3.13 (P13); no longer JP2.1, R12.2
- net LINK_CURR: now also J3.4 (P4)
- net PB7: now also J3.7 (P7)
- net PE2: now also J3.11 (P11)
- net PE3: now also J3.9 (P9)
- net YLW_DRVH_R: now also TP14.1
- net YLW_DRVL_R: now also TP15.1
- net YLW_H: now also TP8.1
- net YLW_L: now also TP9.1
Other:
- moved on the sheet: C1, C10, C11, C12, C13, C14, C15, C16, C17, C18, C19, C2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
