File: Hardware/Three_Phase_Inverter_Controller.sch (KiCad schematic (older format))
At the start: 152 parts, among them J1 POWER, J2 HALL, J3 IN/I2C, J4 UART, J5 USB_B, J6 ISP, Q1 IXFN110N60P3, Q2 IXFN110N60P3, Q3 IXFN110N60P3, Q4 IXFN110N60P3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

Commit message: Generate dimension check PDF
Parts:
- J3: footprint (none) -> Pin_Headers:Pin_Header_Angled_2x08_Pitch2.54mm
Connections:
- net CMD_CURR0: now also J3.9 (P9); no longer J3.8 (P8)
- net CMD_CURR1: now also J3.7 (P7); no longer J3.10 (P10)
- net CMD_CURR2: now also J3.5 (P5); no longer J3.12 (P12)
- net CMD_CURR3: now also J3.3 (P3); no longer J3.14 (P14)
- net CMD_CURR4: now also J3.1 (P1); no longer J3.16 (P16)
- net GND: now also J3.11 (P11), J3.12 (P12), J3.14 (P14), J3.15 (P15), J3.16 (P16); no longer J3.1 (P1), J3.2 (P2), J3.3 (P3), J3.5 (P5), J3.6 (P6)
- net I2C_SCL: now also J3.2 (P2); no longer J3.15 (P15)
- net I2C_SDA: now also J3.4 (P4); no longer J3.13 (P13)
- net LINK_CURR: now also J3.13 (P13); no longer J3.4 (P4)
- net PB7: now also J3.10 (P10); no longer J3.7 (P7)
- net PE2: now also J3.6 (P6); no longer J3.11 (P11)
- net PE3: now also J3.8 (P8); no longer J3.9 (P9)

Commit message: Did stuff
Connections:
- net +12V: no longer TP4.1
- net VIN: now also TP4.1
Other:
- moved on the sheet: R45, TP4
Changed lines of the file:
@@
 EESchema Schematic File Version 2
-LIBS:Three_Phase_Inverter_Controller-rescue
 LIBS:power
 LIBS:device
@@
 L R_Small R45
 U 1 1 591E717E
-P 2725 1450
-F 0 "R45" V 2650 1375 50  0000 L CNN
-F 1 "0.05R" V 2800 1350 50  0000 L CNN
-F 2 "Resistors_SMD:R_1206" H 2725 1450 50  0001 C CNN
-F 3 "" H 2725 1450 50  0001 C CNN
-	1    2725 1450
+P 2975 1450
+F 0 "R45" V 2900 1375 50  0000 L CNN
+F 1 "0.05R" V 3050 1350 50  0000 L CNN
+F 2 "Resistors_SMD:R_1206" H 2975 1450 50  0001 C CNN
+F 3 "" H 2975 1450 50  0001 C CNN
+	1    2975 1450
 	0    1    1    0
 $EndComp
@@
 Connection ~ 4450 1450
 Wire Wire Line
-	2375 1450 2625 1450
+	2375 1450 2875 1450
 Wire Wire Line
 	4450 1775 4450 1950
@@
 	7125 3825 7125 4075
 Wire Wire Line
-	2825 1450 4000 1450
+	3075 1450 4000 1450
 Connection ~ 3375 1450
 Text Label 2400 1450 0    47   ~ 0
@@
 L TEST TP4
 U 1 1 5921A38A
-P 3000 1400
-F 0 "TP4" H 3078 1540 50  0000 L CNN
-F 1 "VIN" H 3078 1449 50  0000 L CNN
-F 2 "Measurement_Points:Test_Point_Keystone_5019_Minature" H 3000 1400 50  0001 C CNN
-F 3 "" H 3000 1400 50  0001 C CNN
-	1    3000 1400
+P 2700 1400
+F 0 "TP4" H 2525 1600 50  0000 L CNN
+F 1 "VIN" H 2525 1525 50  0000 L CNN
+F 2 "Measurement_Points:Test_Point_Keystone_5019_Minature" H 2700 1400 50  0001 C CNN
+F 3 "" H 2700 1400 50  0001 C CNN
+	1    2700 1400
 	1    0    0    -1
 $EndComp
 Wire Wire Line
-	3000 1400 3000 1450
-Connection ~ 3000 1450
+	2700 1400 2700 1450
 Text Notes 8850 5125 0    47   ~ 0
 Trip point (Low to High): 10.628 VDC (12V_HLDP)\nTrip point (High to Low): 10.773 VDC (12V_HLDP)
@@
 Wire Wire Line
 	1200 8725 1200 10650
+Connection ~ 2700 1450
 $EndSCHEMATC

Commit message: Started layout. Minor adjustments to schematic to make layout easier.
Parts:
- removed D3: LNJ167W8RRA, symbol LED_Dual
- added D3, D7: GREEN, LEDs:LED_1206, symbol LED_ALT
- added D8: RED, LEDs:LED_1206, symbol LED_ALT
- added Q7: BSS806NE, TO_SOT_Packages_SMD:SOT-23, symbol Q_NMOS_GSD
- added R39: 180R, Resistors_SMD:R_0603, symbol R_Small
- L1: footprint (none) -> FritzLib:BOURNS_SDR0604
- U7: footprint Housings_DFN_QFN:DFN-8-1EP_3x3mm_Pitch0.5mm -> Housings_DFN_QFN:DFN-10-1EP_3x3mm_Pitch0.5mm
Connections:
- net +5V: now also D3.2 (A), D7.2 (A), D8.2 (A)
- net GND: now also Q7.2 (S)
- net at R30.1: now also D8.1 (K)
- net at R29.1: now also D3.1 (K)
- net PB7 renamed ULED
- net ULED: now also Q7.1 (G)
- new net: Q7.3 (D), R39.1
- new net: D7.1 (K), R39.2
Other:
- moved on the sheet: C24, C25, C26, C27, C28, C29, C30, R27, R31, R46, SW1, U7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

Commit message: More routing and component placement complete
Connections:
- net YLED renamed RLED
