File: Hardware/_autosave-Three_Phase_Inverter_Controller.kicad_pcb (KiCad board)
At the start: 2 copper layers, 152.4 x 127 mm, 141 parts, among them J1 POWER, J2 HALL, J3 CURRENT, J4 I2C, J5 SPARE, J6 UART, J7 USB_B, J8 ISP, Q1 IXFN110N60P3, Q2 IXFN110N60P3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

Commit message: Changed connector, started layout, save before reloading new netlist
Parts:
- added D1: PMEG6030ETP, FritzLib:SOD-128, F.Cu at (92.7, 35.6)
- added D2: PMEG6030ETP, FritzLib:SOD-128, F.Cu at (-452.0, -27.6)
- added D4: PMEG6030ETP, FritzLib:SOD-128, F.Cu at (-445.8, -30.8)
- added D5: PMEG6030ETP, FritzLib:SOD-128, F.Cu at (-452.0, -24.4)
- added D6: PMEG6030ETP, FritzLib:SOD-128, F.Cu at (-445.8, -27.6)
- moved C4 617.8 mm to (104.1, 50.8)
- moved C3 607.8 mm to (104.1, 38.1)
- moved C5 599.3 mm to (88.9, 45.7), turned to 180 degrees
- moved R45 528.7 mm to (86.4, 35.6), turned to 180 degrees
- moved C1 511.1 mm to (76.2, 43.2), turned to 270 degrees
- moved J2 14.4 mm to (76.2, 104.1)
- moved J3 11.4 mm to (81.3, 99.1)
- moved J4 11.4 mm to (81.3, 63.5)
- moved J5 11.4 mm to (81.3, 76.2)
- moved J6 11.4 mm to (81.3, 124.5)
- moved J7 10.2 mm to (71.1, 140.3)
- moved J1 5.08 mm to (76.2, 35.6)
Connections:
- C15 pad 1: +5V -> +3V3_FTDI
- C26 pad 1: +5V -> +5V_USB
- C3 pad 1: +5V -> +12V_HLDP
- C37 pad 1: +5V -> +12V_HLDP
- C38 pad 1: +5V -> +12V_HLDP
- C39 pad 1: +5V -> +12V_HLDP
- C4 pad 1: +5V -> +12V_HLDP
- C40 pad 1: +5V -> +12V_HLDP
- C41 pad 1: +5V -> +12V_HLDP
- C42 pad 1: +5V -> +12V_HLDP
- C44 pad 1: +5V -> +5V_USB
- C5 pad 1: +5V -> +12V_HLDP
- C6 pad 1: +5V -> +12V_HLDP
- C7 pad 1: +5V -> +12V_HLDP
- C9 pad 1: +5V -> +12V_HLDP
- J7 pad 1: +5V -> +5V_USB
- R7 pad 2: +5V -> +5V_USB
- TP6 pad 1: +5V -> +12V_HLDP
- TVS1 pad 4: +5V -> +5V_USB
- U1 pad 1: +5V -> +12V_HLDP
- U10 pad 3: +5V -> +12V_HLDP
- U11 pad 3: +5V -> +12V_HLDP
- U2 pad 2: +5V -> +12V_HLDP
- U2 pad 3: +5V -> +12V_HLDP
- U4 pad 10: +5V -> +3V3_FTDI
- U4 pad 11: +5V -> +3V3_FTDI
- U4 pad 3: +5V -> +3V3_FTDI
- U7 pad 5: +5V -> +5V_USB
- U9 pad 3: +5V -> +12V_HLDP
Other:
- rule pad_to_mask_clearance: 0.2 -> 0.0508
