File: Hardware/_autosave-Three_Phase_Inverter_Controller.kicad_pcb (KiCad board)
At the start: 2 copper layers, 165.1 x 127 mm, 150 parts, among them J1 POWER, J2 HALL, J3 IN/I2C, J4 UART, J5 USB_B, J6 ISP, Q1 IXFN110N60P3, Q2 IXFN110N60P3, Q3 IXFN110N60P3, Q4 IXFN110N60P3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

Commit message: Started layout. Minor adjustments to schematic to make layout easier.
Parts:
- U7: footprint Housings_DFN_QFN:DFN-8-1EP_3x3mm_Pitch0.5mm -> Housings_DFN_QFN:DFN-10-1EP_3x3mm_Pitch0.5mm
- moved TP7 564.6 mm to (87.0, 59.1)
- moved C26 538.5 mm to (78.1, 70.5), turned to 180 degrees
- moved C28 533.1 mm to (86.4, 68.6)
- moved R46 528.7 mm to (84.5, 63.5), turned to 270 degrees
- moved C11 403.9 mm to (-49.5, 26.0), turned to 270 degrees
- moved R18 400.3 mm to (-41.3, 36.2), turned to 90 degrees
- moved R19 392.3 mm to (-39.5, 36.2), turned to 90 degrees
- moved R16 374.5 mm to (-51.4, 26.0), turned to 270 degrees
- moved U7 203.1 mm to (80.5, 66.8), turned to 0 degrees
- moved U3 67.2 mm to (-34.8, 31.4), turned to 180 degrees
- moved C21 1.91 mm to (82.3, 56.9)
- moved C43 1.91 mm to (71.0, 48.4)
- moved C7 1.91 mm to (89.3, 52.2)
- moved C9 1.91 mm to (87.0, 51.6)
- moved D2 1.91 mm to (77.4, 55.0)
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Routing:
- net +5V_BUCK: track 29.1 -> 47.4 mm
- net +12V_HLDP: track 61.8 -> 59.3 mm
