File: Hardware/Three_Phase_Inverter_Controller.kicad_pcb (KiCad board)
At the start: 2 copper layers, 152.4 x 127 mm, 141 parts, among them J1 POWER, J2 HALL, J3 CURRENT, J4 I2C, J5 SPARE, J6 UART, J7 USB_B, J8 ISP, Q1 IXFN110N60P3, Q2 IXFN110N60P3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

Commit message: More layout done
Parts:
- removed J7: USB_B, FritzLib:USB-B_62910416121
- removed J8: ISP, Pin_Headers:Pin_Header_Straight_2x03_Pitch2.54mm
- added D1: PMEG6030ETP, FritzLib:SOD-128, F.Cu at (90.2, 35.6)
- added D2: PMEG6030ETP, FritzLib:SOD-128, F.Cu at (-452.0, -27.6)
- added D4: PMEG6030ETP, FritzLib:SOD-128, F.Cu at (-445.8, -30.8)
- added D5: PMEG6030ETP, FritzLib:SOD-128, F.Cu at (-452.0, -24.4)
- added D6: PMEG6030ETP, FritzLib:SOD-128, F.Cu at (-445.8, -27.6)
- J3: value CURRENT -> IN/I2C; footprint Pin_Headers:Pin_Header_Angled_1x08_Pitch2.54mm -> Pin_Headers:Pin_Header_Angled_2x08_Pitch2.54mm
- J4: value I2C -> UART
- J5: value SPARE -> USB_B; footprint Pin_Headers:Pin_Header_Angled_1x04_Pitch2.54mm -> FritzLib:USB-B_62910416121
- J6: value UART -> ISP; footprint Pin_Headers:Pin_Header_Angled_1x04_Pitch2.54mm -> Pin_Headers:Pin_Header_Straight_2x03_Pitch2.54mm
- moved C4 615.3 mm to (101.6, 50.8)
- moved C3 605.3 mm to (101.6, 38.1)
- moved C5 596.8 mm to (86.4, 45.7), turned to 180 degrees
- moved U2 575.7 mm to (89.5, 59.0)
- moved U7 558.6 mm to (104.6, 61.6)
- moved U1 557.7 mm to (95.4, 64.5)
- moved R45 526.2 mm to (83.8, 35.6), turned to 180 degrees
- moved C1 517.3 mm to (83.8, 38.1), turned to 180 degrees
- moved J6 61.1 mm to (129.5, 71.1)
- moved J4 53.6 mm to (81.3, 106.7)
- moved J3 53.4 mm to (83.8, 142.2)
- moved U4 46.3 mm to (96.5, 84.1), turned to 90 degrees
- moved J5 23.9 mm to (71.1, 84.4), turned to 270 degrees
- moved J2 20.5 mm to (76.2, 111.8)
- moved J1 5.08 mm to (76.2, 35.6)
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Connections:
- net PGOOD renamed /PGOOD
- C15 pad 1: +5V -> +3V3_FTDI
- C26 pad 1: +5V -> +5V_USB
- C3 pad 1: +5V -> +12V_HLDP
- C37 pad 1: +5V -> +12V_HLDP
- C38 pad 1: +5V -> +12V_HLDP
- C39 pad 1: +5V -> +12V_HLDP
- C4 pad 1: +5V -> +12V_HLDP
- C40 pad 1: +5V -> +12V_HLDP
- C41 pad 1: +5V -> +12V_HLDP
- C42 pad 1: +5V -> +12V_HLDP
- C44 pad 1: +5V -> +5V_USB
- C5 pad 1: +5V -> +12V_HLDP
- C6 pad 1: +5V -> +12V_HLDP
- C7 pad 1: +5V -> +12V_HLDP
- C9 pad 1: +5V -> +12V_HLDP
- J3 pad 1: /CMD_CURR4 -> GND
- J3 pad 2: /CMD_CURR3 -> GND
- J3 pad 3: /CMD_CURR2 -> GND
- J3 pad 4: /CMD_CURR1 -> /LINK_CURR
- J3 pad 5: /CMD_CURR0 -> GND
- J3 pad 7: /LINK_CURR -> /PB7
- J3 pad 8: GND -> /CMD_CURR0
- J4 pad 2: /I2C_SCL -> /RXD
- J4 pad 3: /I2C_SDA -> /TXD
- J5 pad 1: GND -> +5V_USB
- J5 pad 2: /PB7 -> /USB-
- J5 pad 3: /PE3 -> /USB+
- J5 pad 4: /PE2 -> GND
- J6 pad 1: GND -> /PB4/MISO
- J6 pad 2: /RXD -> +5V
- J6 pad 3: /TXD -> /SHDN/SCK
- J6 pad 4: GND -> /MODE/MOSI
- JP2 pad 1: /I2C_SDA -> /I2C_SCL
- JP3 pad 1: /I2C_SCL -> /I2C_SDA
- R12 pad 2: /I2C_SDA -> /I2C_SCL
- R13 pad 2: /I2C_SCL -> /I2C_SDA
- R7 pad 2: +5V -> +5V_USB
- TP6 pad 1: +5V -> +12V_HLDP
- TVS1 pad 4: +5V -> +5V_USB
- U1 pad 1: +5V -> +12V_HLDP
- U10 pad 3: +5V -> +12V_HLDP
- U11 pad 3: +5V -> +12V_HLDP
- U2 pad 2: +5V -> +12V_HLDP
- U2 pad 3: +5V -> +12V_HLDP
- U4 pad 10: +5V -> +3V3_FTDI
- U4 pad 11: +5V -> +3V3_FTDI
- U4 pad 3: +5V -> +3V3_FTDI
- U7 pad 5: +5V -> +5V_USB
- U9 pad 3: +5V -> +12V_HLDP
Other:
- rule pad_to_mask_clearance: 0.2 -> 0.0508

Commit message: Generate dimension check PDF
Parts:
- moved U6 585.3 mm to (78.6, 62.9)
- moved TVS1 580.2 mm to (96.5, 83.8)
- moved U3 553.7 mm to (85.1, 63.5)
- moved J6 121.2 mm to (118.1, 191.8)
- moved U2 52.3 mm to (139.9, 45.1)
- moved U5 20.5 mm to (137.2, 108.0)
- moved U7 18.1 mm to (122.0, 66.3), turned to 180 degrees
- moved U4 9.21 mm to (105.7, 84.1)
- moved U1 4.09 mm to (91.4, 63.5)
- moved C4 3.96 mm to (102.7, 47.0)
- moved C5 2.84 mm to (88.9, 47.0)
- moved C3 2.84 mm to (102.9, 35.6)
- moved J1 1.91 mm to (74.3, 35.6)
- moved J2 1.91 mm to (74.3, 111.8)
- moved D1 1.27 mm to (91.4, 35.6)
Connections:
- C21 pad 1: +5V -> +5V_BUCK
- C25 pad 1: +5V -> +5V_BUCK
- C43 pad 1: +5V -> +5V_BUCK
- J3 pad 1: GND -> /CMD_CURR4
- J3 pad 10: /CMD_CURR1 -> /PB7
- J3 pad 11: /PE2 -> GND
- J3 pad 12: /CMD_CURR2 -> GND
- J3 pad 13: /I2C_SDA -> /LINK_CURR
- J3 pad 14: /CMD_CURR3 -> GND
- J3 pad 15: /I2C_SCL -> GND
- J3 pad 16: /CMD_CURR4 -> GND
- J3 pad 2: GND -> /I2C_SCL
- J3 pad 3: GND -> /CMD_CURR3
- J3 pad 4: /LINK_CURR -> /I2C_SDA
- J3 pad 5: GND -> /CMD_CURR2
- J3 pad 6: GND -> /PE2
- J3 pad 7: /PB7 -> /CMD_CURR1
- J3 pad 8: /CMD_CURR0 -> /PE3
- J3 pad 9: /PE3 -> /CMD_CURR0
- R25 pad 1: +5V -> +5V_BUCK
- R27 pad 1: +5V -> +5V_BUCK
- R46 pad 1: +5V -> +5V_BUCK
- TP7 pad 1: +5V -> +5V_BUCK
- U7 pad 1: +5V -> +5V_BUCK

Commit message: Updated BOM?
Parts:
- moved J4 1.27 mm to (81.3, 105.4)
- moved J3 1.27 mm to (83.8, 143.5)
Changed lines of the file:
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@@
     (visible_elements 7FFDEFFF)
     (pcbplotparams
-      (layerselection 0x00030_ffffffff)
+      (layerselection 0x0d030_ffffffff)
       (usegerberextensions false)
       (excludeedgelayer true)
@@
       (padsonsilk false)
       (subtractmaskfromsilk false)
-      (outputformat 1)
+      (outputformat 4)
       (mirror false)
-      (drillshape 1)
+      (drillshape 0)
       (scaleselection 1)
       (outputdirectory ""))
@@
     (add_net "Net-(U8-Pad1)")
   )
+  (module FritzLib:USB-B_62910416121 (layer F.Cu)
+    (at 71.12 84.405 270)
+    (fp_text reference J5 (at 0 -6 270) (layer F.SilkS)
+      (effects (font (size 1 1) (thickness 0.15)))
+    )
+    (fp_text value USB_B (at 0 2 270) (layer F.Fab)
+      (effects (font (size 1 1) (thickness 0.15)))
+    )
+    (fp_line (start -6 -2) (end -6 -2) (layer F.SilkS) (width 0.15))
+    (fp_line (start -6 -6) (end -6 -2) (layer F.SilkS) (width 0.15))
+    (fp_line (start 6 -2) (end 6 -2) (layer F.SilkS) (width 0.15))
+    (fp_line (start 6 -6) (end 6 -2) (layer F.SilkS) (width 0.15))
+    (fp_line (start 6 -13) (end 6 -13) (layer F.SilkS) (width 0.15))
+    (fp_line (start 6 -15) (end 6 -13) (layer F.SilkS) (width 0.15))
+    (fp_line (start 3 -15) (end 6 -15) (layer F.SilkS) (width 0.15))
+    (fp_line (start -3 -15) (end -3 -15) (layer F.SilkS) (width 0.15))
+    (fp_line (start -6 -15) (end -3 -15) (layer F.SilkS) (width 0.15))
+    (fp_line (start -6 -13) (end -6 -15) (layer F.SilkS) (width 0.15))
+    (fp_line (start -6.2 0) (end 6.2 0) (layer Eco2.User) (width 0.15))
+    (pad 5 smd rect (at -7 -9.58 270) (size 5 6.4) (layers F.Cu F.Paste F.Mask)
+      (net 3 "Net-(C2-Pad2)"))
+    (pad "" np_thru_hole circle (at 2.75 -9 270) (size 1.3 1.3) (drill 1.3) (layers *.Cu *.Mask))
+    (pad "" np_thru_hole circle (at -2.75 -9 270) (size 1.3 1.3) (drill 1.3) (layers *.Cu *.Mask))
+    (pad 4 smd rect (at -1.875 -16 270) (size 0.7 3) (layers F.Cu F.Paste F.Mask)
+      (net 1 GND))
+    (pad 3 smd rect (at 0.625 -16 270) (size 0.7 3) (layers F.Cu F.Paste F.Mask)
+      (net 53 /USB+))
+    (pad 1 smd rect (at 1.875 -16 270) (size 0.7 3) (layers F.Cu F.Paste F.Mask)
+      (net 89 +5V_USB))
+    (pad 2 smd rect (at -0.625 -16 270) (size 0.7 3) (layers F.Cu F.Paste F.Mask)
+      (net 54 /USB-))
+    (pad 5 smd rect (at 7 -9.58 270) (size 5 6.4) (layers F.Cu F.Paste F.Mask)
+      (net 3 "Net-(C2-Pad2)"))
+    (model C:/Users/jfrit/Documents/GitHub/Kicad_Lib/3D_Source/STEP-62910416121-rev1.stp
+      (at (xyz 0 0.32 0.23))
+      (scale (xyz 1 1 1))
+      (rotate (xyz 0 0 0))
+    )
+  )
   (module Capacitors_SMD:C_0603 (layer F.Cu)
     (at 83.82 38.1 180)
@@
   )
   (module Pin_Headers:Pin_Header_Angled_1x04_Pitch2.54mm (layer F.Cu)
-    (at 81.28 106.68 180)
+    (at 81.28 105.41 180)
     (descr "Through hole angled pin header, 1x04, 2.54mm pitch, 6mm pin length, single row")
     (tags "Through hole angled pin header THT 1x04 2.54mm single row")
@@
   )
   (module Pin_Headers:Pin_Header_Angled_2x08_Pitch2.54mm (layer F.Cu)
-    (at 83.82 142.24 180)
+    (at 83.82 143.51 180)
     (descr "Through hole angled pin header, 2x08, 2.54mm pitch, 6mm pin length, double rows")
     (tags "Through hole angled pin header THT 2x08 2.54mm double row")
@@
     )
   )
-  (module FritzLib:USB-B_62910416121 (layer F.Cu)
-    (at 71.12 84.405 270)
-    (fp_text reference J5 (at 0 -6 270) (layer F.SilkS)
-      (effects (font (size 1 1) (thickness 0.15)))
-    )
-    (fp_text value USB_B (at 0 2 270) (layer F.Fab)
-      (effects (font (size 1 1) (thickness 0.15)))
-    )
-    (fp_line (start -6.2 0) (end 6.2 0) (layer Eco2.User) (width 0.15))
-    (fp_line (start -6 -13) (end -6 -15) (layer F.SilkS) (width 0.15))
-    (fp_line (start -6 -15) (end -3 -15) (layer F.SilkS) (width 0.15))
-    (fp_line (start -3 -15) (end -3 -15) (layer F.SilkS) (width 0.15))
-    (fp_line (start 3 -15) (end 6 -15) (layer F.SilkS) (width 0.15))
-    (fp_line (start 6 -15) (end 6 -13) (layer F.SilkS) (width 0.15))
-    (fp_line (start 6 -13) (end 6 -13) (layer F.SilkS) (width 0.15))
-    (fp_line (start 6 -6) (end 6 -2) (layer F.SilkS) (width 0.15))
-    (fp_line (start 6 -2) (end 6 -2) (layer F.SilkS) (width 0.15))
-    (fp_line (start -6 -6) (end -6 -2) (layer F.SilkS) (width 0.15))
-    (fp_line (start -6 -2) (end -6 -2) (layer F.SilkS) (width 0.15))
-    (pad 5 smd rect (at 8 -9.58 270) (size 5 6.4) (layers F.Cu F.Paste F.Mask)
-      (net 3 "Net-(C2-Pad2)"))
-    (pad 2 smd rect (at -0.625 -16 270) (size 0.7 3) (layers F.Cu F.Paste F.Mask)
-      (net 54 /USB-))
-    (pad 1 smd rect (at 1.875 -16 270) (size 0.7 3) (layers F.Cu F.Paste F.Mask)
-      (net 89 +5V_USB))
-    (pad 3 smd rect (at 0.625 -16 270) (size 0.7 3) (layers F.Cu F.Paste F.Mask)
-      (net 53 /USB+))
-    (pad 4 smd rect (at -1.875 -16 270) (size 0.7 3) (layers F.Cu F.Paste F.Mask)
-      (net 1 GND))
-    (pad "" np_thru_hole circle (at -2.75 -9 270) (size 1.3 1.3) (drill 1.3) (layers *.Cu *.Mask))
-    (pad "" np_thru_hole circle (at 2.75 -9 270) (size 1.3 1.3) (drill 1.3) (layers *.Cu *.Mask))
-    (pad 5 smd rect (at -8 -9.58 270) (size 5 6.4) (layers F.Cu F.Paste F.Mask)
-      (net 3 "Net-(C2-Pad2)"))
-    (model C:/Users/jfrit/Documents/GitHub/Kicad_Lib/3D_Source/STEP-62910416121-rev1.stp
-      (at (xyz 0 0.32 0.23))
-      (scale (xyz 1 1 1))
-      (rotate (xyz 0 0 0))
-    )
-  )

Commit message: Did stuff
Parts:
- moved TP4 564.6 mm to (85.1, 31.8)
- moved U2 303.9 mm to (-164.1, 43.4)
- moved C21 303.3 mm to (-166.5, 34.5), turned to 270 degrees
- moved R26 298.8 mm to (-158.9, 44.7), turned to 90 degrees
- moved D2 297.9 mm to (-161.5, 38.3)
- moved R25 297.2 mm to (-157.0, 44.7), turned to 270 degrees
- moved C24 296.5 mm to (-158.9, 47.9), turned to 270 degrees
- moved C7 295.0 mm to (-173.5, 40.9), turned to 90 degrees
- moved R27 293.3 mm to (-157.0, 47.9), turned to 90 degrees
- moved R17 279.3 mm to (-166.5, 47.2)
- moved C9 278.8 mm to (-171.0, 41.5), turned to 90 degrees
- moved C43 271.1 mm to (-169.1, 39.0), turned to 270 degrees
- moved C16 225.8 mm to (-209.7, 8.26)
- moved U7 160.6 mm to (-35.4, 34.5)
- moved U1 108.0 mm to (-11.4, 30.5)
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Connections:
- TP4 pad 1: +12V -> /VIN
Other:
- rule trace_min: 0.2 -> 0.1524
- board text added: "TODO Flip schottkey diode schematic symbol around (anode should be pin 1, cathode should be pin 2)"

Commit message: Started layout. Minor adjustments to schematic to make layout easier.
Parts:
- added D3: GREEN, LEDs:LED_1206, F.Cu at (-265.6, -50.6)
- added D7: GREEN, LEDs:LED_1206, F.Cu at (-259.9, -50.6)
- added D8: RED, LEDs:LED_1206, F.Cu at (-265.6, -45.2)
- added L1: 68uH, FritzLib:BOURNS_SDR0604, F.Cu at (72.1, 54.0)
- added Q7: BSS806NE, TO_SOT_Packages_SMD:SOT-23, F.Cu at (-272.6, -49.7)
- added R39: 180R, Resistors_SMD:R_0603, F.Cu at (-274.6, -43.7)
- moved TP7 564.6 mm to (87.0, 59.1)
- moved TP5 545.0 mm to (54.6, 32.4)
- moved TP6 517.2 mm to (41.3, 41.3), turned to 90 degrees
- moved C11 403.9 mm to (-49.5, 26.0), turned to 270 degrees
- moved R18 400.3 mm to (-41.3, 36.2), turned to 90 degrees
- moved R19 392.3 mm to (-39.5, 36.2), turned to 90 degrees
- moved C10 389.0 mm to (-51.4, 29.2), turned to 270 degrees
- moved R16 374.5 mm to (-51.4, 26.0), turned to 270 degrees
- moved C6 373.3 mm to (-58.4, 26.0), turned to 270 degrees
- moved C16 298.0 mm to (85.0, 53.0), turned to 270 degrees
- moved C7 263.1 mm to (89.3, 52.2), turned to 270 degrees
- moved C9 258.2 mm to (87.0, 51.6), turned to 270 degrees
- moved C21 249.9 mm to (82.3, 56.9), turned to 90 degrees
- moved R17 248.9 mm to (82.3, 45.9), turned to 180 degrees
- moved U2 244.0 mm to (79.9, 49.7), turned to 180 degrees
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Connections:
- net /PB7 renamed /ULED
Routing:
- net GND: track 0.00 -> 62.3 mm, vias 0 -> 1
- net +12V_HLDP: track 0.00 -> 59.3 mm
- net +5V_BUCK: track 0.00 -> 47.4 mm, vias 0 -> 2
- net +12V: track 0.00 -> 15.1 mm
- net /VIN: track 0.00 -> 10.6 mm
- net /PGOOD: track 0.00 -> 8.61 mm
- net /BUCK_SW: track 0.00 -> 8.09 mm, vias 0 -> 2
- net /BUCK_FB: track 0.00 -> 6.24 mm
- net /BUCK_B: track 0.00 -> 2.65 mm
- net Net-(R17-Pad1): track 0.00 -> 2.18 mm
- added copper zone on F.Cu, net +12V_HLDP
- added copper zone on F.Cu, net +5V_BUCK
- added copper zone on F.Cu, net /BUCK_SW
- added copper zone on F.Cu, net GND
Other:
- board size 152.4 x 127 mm -> 165.1 x 127 mm
- rule via_min_size: 0.4 -> 0.4064
- board text removed: "TODO Flip schottkey diode schematic symbol around (anode should be pin 1, cathode should be pin 2)"

Commit message: More routing and component placement complete
Parts:
- U7: footprint Housings_DFN_QFN:DFN-8-1EP_3x3mm_Pitch0.5mm -> Housings_DFN_QFN:DFN-10-1EP_3x3mm_Pitch0.5mm
- moved C25 565.3 mm to (85.1, 66.0)
- moved C26 544.7 mm to (85.1, 68.6)
- moved R46 528.7 mm to (84.5, 63.5), turned to 270 degrees
- moved C29 523.3 mm to (73.0, 68.6), turned to 270 degrees
- moved C28 522.8 mm to (75.6, 68.6), turned to 270 degrees
- moved C13 519.4 mm to (57.7, 59.7), turned to 180 degrees
- moved C19 505.4 mm to (53.7, 55.9), turned to 180 degrees
- moved R23 502.9 mm to (48.6, 59.1), turned to 90 degrees
- moved R29 502.8 mm to (50.2, 54.6), turned to 270 degrees
- moved R30 502.3 mm to (46.4, 54.6), turned to 270 degrees
- moved R22 500.4 mm to (51.1, 61.6), turned to 180 degrees
- moved R24 483.3 mm to (50.5, 59.1), turned to 270 degrees
- moved D3 329.5 mm to (48.9, 47.6), turned to 180 degrees
- moved D8 327.2 mm to (48.9, 45.1), turned to 180 degrees
- moved U7 202.3 mm to (79.7, 66.8)
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Connections:
- U7 pad 1: +5V_BUCK -> +5V_USB
- U7 pad 5: +5V_USB -> +5V_BUCK
Routing:
- net +12V_HLDP: track 59.3 -> 49.7 mm
- net +5V_BUCK: track 47.4 -> 45.5 mm

Commit message: Add new 3D models/Routed more
Parts:
- moved JP5 22.1 mm to (-85.7, 88.3)
- moved JP1 18.6 mm to (-85.8, 107.3)
- moved J6 14.5 mm to (121.9, 177.8)
- moved JP4 14.0 mm to (-85.7, 102.9)
- moved JP3 12.1 mm to (-85.8, 98.4)
- moved TP12 2.14 mm to (-514.4, -106.7)
Connections:
- net /YLED renamed /RLED

Commit message: Finished initial component placement
Parts:
- removed R3k1: 10k, Resistors_SMD:R_0603
- added R47: 10k, Resistors_SMD:R_0603, F.Cu at (177.8, 44.5)
- TP1, TP10, TP11, TP12, TP13, TP14, TP15, TP16, TP17, TP18, TP19, TP2, TP3, TP4, TP5, TP6, TP7, TP8, TP9: footprint Measurement_Points:Test_Point_Keystone_5019_Minature -> FritzLib:Test_Point_Keystone_5019_Minature
- U10, U11, U9: footprint Housings_SOIC:SOIC-16W_7.5x10.3mm_Pitch1.27mm -> FritzLib:SOIC-16W_7.5x10.3mm_Pitch1.27mm
- moved TP15 738.0 mm to (177.8, 142.2)
- moved TP17 730.7 mm to (158.8, 142.2)
- moved TP14 714.9 mm to (177.8, 35.6)
- moved TP16 704.2 mm to (158.8, 35.6)
- moved TP8 696.7 mm to (144.8, 96.5)
- moved TP9 692.7 mm to (144.8, 101.6)
- moved TP11 684.7 mm to (144.8, 91.4)
- moved TP19 684.1 mm to (114.3, 142.2)
- moved TP12 684.0 mm to (144.8, 76.2)
- moved TP10 682.2 mm to (144.8, 86.4)
- moved TP13 675.6 mm to (144.8, 81.3)
- moved R34 663.2 mm to (177.8, 134.0), turned to 180 degrees
- moved TP18 659.5 mm to (114.3, 35.6)
- moved C35 649.3 mm to (168.9, 81.5), turned to 90 degrees
- moved C36 641.9 mm to (168.9, 62.5), turned to 90 degrees
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Connections:
- J6 pad 1: /PB4/MISO -> /M_SD/MISO
- J6 pad 3: /SHDN/SCK -> /EX_SD/SCK
Routing:
- net GND: track 62.3 -> 61.2 mm, vias 1 -> 0
- net (no net): track 0.00 -> 1.16 mm, vias 0 -> 1
Other:
- board text added: "A"
- board text added: "B"
- board text added: "C"
- board text added: "CC0"
- board text added: "CC1"
- board text added: "CC2"
- board text added: "CC3"
- board text added: "CC4"
- board text added: "GND"
- board text added: "LKC"
- board text added: "PB6"
- board text added: "PE2"
- board text added: "PE3"
- board text added: "RXD"
- board text added: "SCL"
- board text added: "SDA"
- board text added: "TXD"
